File: Kicad/BEM.kicad_sch (KiCad schematic)
At the start: 17 parts, among them U2 ACS712xLCTR-30A, U3 ACS712xLCTR-30A, U4 ACS712xLCTR-30A, U5 ACS712xLCTR-30A

Commit message: Added: Schem V2, Schem.png
Parts:
- added J2: SD_Card_Device, symbol Connector:SD_Card_Device
Connections:
- net A: now also U1.24 (ADC2_CH2/GPIO2); no longer U1.14 (MTDI/GPIO12/ADC2_CH5)
- net A1: now also U1.8 (32K_XP/GPIO32/ADC1_CH4); no longer U1.29 (GPIO5)
- net B: now also U1.26 (ADC2_CH0/GPIO4); no longer U1.16 (MTCK/GPIO13/ADC2_CH4)
- net B1: now also U1.4 (SENSOR_VP/GPIO36/ADC1_CH0); no longer U1.27 (GPIO16)
- net C: now also U1.28 (GPIO17); no longer U1.13 (MTMS/GPIO14/ADC2_CH6)
- net C1: now also U1.33 (GPIO21); no longer U1.28 (GPIO17)
- net D: now also U1.5 (SENSOR_VN/GPIO39/ADC1_CH3); no longer U1.23 (MTDO/GPIO15/ADC2_CH3)
- net D1: now also U1.9 (32K_XN/GPIO33/ADC1_CH5); no longer U1.30 (GPIO18)
- net GND: now also J2.2 (GND)
- net INPUT: no longer U1.40 (Vin)
- net at U1.36 (GPIO22): no longer K3.1
- net at U1.37 (GPIO23): now also J2.3 (MOSI); no longer K4.1
- net at U1.31 (GPIO19): now also J2.4 (MISO); no longer K1.1
- net RELAY2: now reaches K2.1
- net RELAY2: now also U1.16 (MTCK/GPIO13/ADC2_CH4); no longer U1.33 (GPIO21)
- new net: J2.6 (CS), U1.29 (GPIO5)
- new net: J2.5 (SCK), U1.30 (GPIO18)
- new net RELAY1: K1.1, U1.14 (MTDI/GPIO12/ADC2_CH5)
- new net RELAY3: K3.1, U1.13 (MTMS/GPIO14/ADC2_CH6)
- new net RELAY4: K4.1, U1.23 (MTDO/GPIO15/ADC2_CH3)
Other:
- note added: "17/11/2024"
- note added: "Better Energy Management (B.E.M.)"
- moved on the sheet: K1, K2, K3, K4, R1, R2, R3, R4, U1, U2, U3, U4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

Commit message: Added: Schem V2, SchemV2.png
Connections:
- net INPUT: now also J2.1 (VCC), U1.40 (Vin)
Changed lines of the file:
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@@
+		)
+	)
+	(global_label "INPUT"
+		(shape input)
+		(at 77.47 170.18 270)
+		(fields_autoplaced yes)
+		(effects
+			(font
+				(size 1.27 1.27)
+			)
+			(justify right)
+		)
+		(property "Intersheetrefs" "${INTERSHEET_REFS}"
+			(at 77.47 178.6686 90)
+			(effects
+				(font
+					(size 1.27 1.27)
+				)
+				(justify right)
+				(hide yes)
+			)
 		)
 	)
@@
 		)
 	)
+	(global_label "INPUT"
+		(shape input)
+		(at 38.1 54.61 0)
+		(fields_autoplaced yes)
+		(effects
+			(font
+				(size 1.27 1.27)
+			)
+			(justify left)
+		)
+		(property "Intersheetrefs" "${INTERSHEET_REFS}"
+			(at 46.5886 54.61 0)
+			(effects
+				(font
+					(size 1.27 1.27)
+				)
+				(justify left)
+				(hide yes)
+			)
+		)
+	)
 	(global_label "B"
 		(shape input)
@@
 				)
 				(justify left)
+				(hide yes)
+			)
+		)
+	)
+	(global_label "INPUT"
+		(shape input)
+		(at 54.61 54.61 180)
+		(fields_autoplaced yes)
+		(effects
+			(font
+				(size 1.27 1.27)
+			)
+			(justify right)
+		)
+		(property "Intersheetrefs" "${INTERSHEET_REFS}"
+			(at 46.1214 54.61 0)
+			(effects
+				(font
+					(size 1.27 1.27)
+				)
+				(justify right)
 				(hide yes)
 			)
@@
 	(symbol
 		(lib_id "power:+5V")
-		(at 52.07 54.61 270)
+		(at 35.56 54.61 270)
 		(unit 1)
 		(exclude_from_sim no)
@@
 		(dnp no)
 		(property "Reference" "#PWR021"
-			(at 48.26 54.61 0)
+			(at 31.75 54.61 0)
 			(effects
 				(font
@@
 		)
 		(property "Value" "+5V"
-			(at 50.038 52.324 90)
+			(at 33.528 52.324 90)
 			(effects
 				(font
@@
 		)
 		(property "Footprint" ""
-			(at 52.07 54.61 0)
+			(at 35.56 54.61 0)
 			(effects
 				(font
@@
 		)
 		(property "Datasheet" ""
-			(at 52.07 54.61 0)
+			(at 35.56 54.61 0)
 			(effects
 				(font
@@
 		)
 		(property "Description" "Power symbol creates a global label with name \"+5V\""
-			(at 52.07 54.61 0)
+			(at 35.56 54.61 0)
 			(effects
 				(font
@@
 					(unit 1)
 				)
-			)
-		)
-	)
-	(symbol
-		(lib_id "power:+5V")
-		(at 77.47 172.72 0)
-		(unit 1)
-		(exclude_from_sim no)
-		(in_bom yes)
-		(on_board yes)
-		(dnp no)
-		(property "Reference" "#PWR025"
-			(at 77.47 176.53 0)
-			(effects
-				(font
-					(size 1.27 1.27)
-				)
-				(hide yes)
-			)
-		)
-		(property "Value" "+5V"
-			(at 75.184 174.752 90)
-			(effects
-				(font
-					(size 1.27 1.27)
-				)
-				(justify left)
-			)
-		)
-		(property "Footprint" ""
-			(at 77.47 172.72 0)
-			(effects
-				(font
-					(size 1.27 1.27)
-				)
-				(hide yes)
-			)
-		)
-		(property "Datasheet" ""
-			(at 77.47 172.72 0)
-			(effects
-				(font
-					(size 1.27 1.27)
-				)
-				(hide yes)
-			)
-		)
-		(property "Description" "Power symbol creates a global label with name \"+5V\""
-			(at 77.47 172.72 0)
-			(effects
-				(font
-					(size 1.27 1.27)
-				)
-				(hide yes)
-			)
-		)
-		(pin "1"
-		)
-		(instances
-			(project "BEM"
-				(path "/39f2b7ab-cdf4-4af2-aee0-3778b0882017"
-					(reference "#PWR025")
-					(unit 1)
-				)

Commit message: Updated: Schematic
Connections:
- net INPUT: now also K1.2, K2.2, K3.2, K4.2
- now unconnected: U1.2 (3V3)
Other:
- moved on the sheet: J2, U1

Commit message: Schematic
Connections:
- net A: now also J2.3 (MOSI), K4.1, U1.10 (DAC_1/ADC2_CH8/GPIO25), U1.11 (DAC_2/ADC2_CH9/GPIO26), U1.36 (GPIO22), U1.37 (GPIO23); no longer U1.24 (ADC2_CH2/GPIO2)
- net A1: now also U1.7 (GPIO35/ADC1_CH7); no longer U1.8 (32K_XP/GPIO32/ADC1_CH4)
- net B: now also U1.12 (ADC2_CH7/GPIO27); no longer U1.26 (ADC2_CH0/GPIO4)
- net B1: now also U1.6 (GPIO34/ADC1_CH6); no longer U1.4 (SENSOR_VP/GPIO36/ADC1_CH0)
- net C: now also U1.8 (32K_XP/GPIO32/ADC1_CH4); no longer U1.28 (GPIO17)
- net C1: now also U1.5 (SENSOR_VN/GPIO39/ADC1_CH3); no longer U1.33 (GPIO21)
- net D: now also U1.9 (32K_XN/GPIO33/ADC1_CH5); no longer U1.5 (SENSOR_VN/GPIO39/ADC1_CH3)
- net D1: now also U1.4 (SENSOR_VP/GPIO36/ADC1_CH0); no longer U1.9 (32K_XN/GPIO33/ADC1_CH5)
- net RELAY1: now also U1.23 (MTDO/GPIO15/ADC2_CH3); no longer U1.14 (MTDI/GPIO12/ADC2_CH5)
- net RELAY2: now also U1.26 (ADC2_CH0/GPIO4); no longer U1.16 (MTCK/GPIO13/ADC2_CH4)
- net RELAY3: now also U1.27 (GPIO16); no longer U1.13 (MTMS/GPIO14/ADC2_CH6)
- removed net RELAY4: K4.1, U1.23 (MTDO/GPIO15/ADC2_CH3)
